Commit message: feat(description): mount PCB and calibrate stylus geometry
- Attach the PCB to base_link and remove its duplicate world model
- Raise the gantry and add four structural support columns
- Add pen-tip collision geometry and update the safe Z travel limits
- Synchronize drawing commands with the revised PCB contact height

File: src/drawbot_description/urdf/drawbot.urdf.xacro (robot description, xacro)
@@ -5,4 +5,10 @@
   <xacro:property name="base_y" value="0.36"/>
   <xacro:property name="base_z" value="0.020"/>
+  <xacro:property name="pcb_x" value="0.25"/>
+  <xacro:property name="pcb_y" value="0.25"/>
+  <xacro:property name="pcb_z" value="0.001"/>
+  <!-- Raise the gantry so joint_pen=0 starts 7.5 mm above the PCB. -->
+  <xacro:property name="gantry_raise" value="0.0195"/>
+  <xacro:property name="support_size" value="0.020"/>
   <xacro:property name="rail_x_len" value="0.32"/>
   <xacro:property name="rail_x_w"   value="0.020"/>
@@ -19,5 +25,6 @@
   <xacro:property name="y_min" value="-0.10"/>
   <xacro:property name="y_max" value="0.10"/>
-  <xacro:property name="z_min" value="-0.025"/>
+  <!-- Tip contact is near -6 mm; allow only 0.5 mm extra compression. -->
+  <xacro:property name="z_min" value="-0.0065"/>
   <xacro:property name="z_max" value="0.020"/>
   <material name="grey"><color rgba="0.45 0.45 0.47 1"/></material>
@@ -26,4 +33,25 @@
   <material name="red"><color rgba="0.85 0.18 0.18 1"/></material>
   <material name="black"><color rgba="0.08 0.08 0.08 1"/></material>
+  <material name="pcb_green"><color rgba="0.04 0.32 0.16 1"/></material>
+  <xacro:macro name="support_column" params="name x y">
+    <link name="${name}">
+      <visual>
+        <geometry><box size="${support_size} ${support_size} ${gantry_raise}"/></geometry>
+        <material name="grey"/>
+      </visual>
+      <collision>
+        <geometry><box size="${support_size} ${support_size} ${gantry_raise}"/></geometry>
+      </collision>
+      <inertial>
+        <mass value="0.05"/>
+        <inertia ixx="0.000003" ixy="0" ixz="0" iyy="0.000003" iyz="0" izz="0.000003"/>
+      </inertial>
+    </link>
+    <joint name="${name}_joint" type="fixed">
+      <parent link="base_link"/>
+      <child link="${name}"/>
+      <origin xyz="${x} ${y} ${base_z + gantry_raise/2}"/>
+    </joint>
+  </xacro:macro>
   <!-- ========== BASE (fixe, horizontale) ========== -->
   <link name="base_link">
@@ -42,4 +70,30 @@
     </inertial>
   </link>
+  <!-- PCB fixée au plateau supérieur du robot -->
+  <link name="pcb_link">
+    <visual>
+      <origin xyz="0 0 ${base_z + pcb_z/2}"/>
+      <geometry><box size="${pcb_x} ${pcb_y} ${pcb_z}"/></geometry>
+      <material name="pcb_green"/>
+    </visual>
+    <collision>
+      <origin xyz="0 0 ${base_z + pcb_z/2}"/>
+      <geometry><box size="${pcb_x} ${pcb_y} ${pcb_z}"/></geometry>
+    </collision>
+    <inertial>
+      <origin xyz="0 0 ${base_z + pcb_z/2}"/>
+      <mass value="0.12"/>
+      <inertia ixx="0.000625" ixy="0" ixz="0" iyy="0.000625" iyz="0" izz="0.00125"/>
+    </inertial>
+  </link>
+  <joint name="pcb_mount_joint" type="fixed">
+    <parent link="base_link"/>
+    <child link="pcb_link"/>
+  </joint>
+  <!-- Colonnes structurelles entre le plateau et les rails relevés -->
+  <xacro:support_column name="support_front_left" x="-0.14" y="0.15"/>
+  <xacro:support_column name="support_front_right" x="0.14" y="0.15"/>
+  <xacro:support_column name="support_back_left" x="-0.14" y="-0.15"/>
+  <xacro:support_column name="support_back_right" x="0.14" y="-0.15"/>
   <!-- Rails X fixes (deux barres horizontales selon X, aux bords Y) -->
   <link name="rail_x_pos">
@@ -60,5 +114,5 @@
     <parent link="base_link"/>
     <child link="rail_x_pos"/>
-    <origin xyz="0 ${base_y/2 - 0.03} ${base_z + rail_x_h/2}"/>
+    <origin xyz="0 ${base_y/2 - 0.03} ${base_z + rail_x_h/2 + gantry_raise}"/>
   </joint>
   <link name="rail_x_neg">
@@ -78,5 +132,5 @@
     <parent link="base_link"/>
     <child link="rail_x_neg"/>
-    <origin xyz="0 ${-base_y/2 + 0.03} ${base_z + rail_x_h/2}"/>
+    <origin xyz="0 ${-base_y/2 + 0.03} ${base_z + rail_x_h/2 + gantry_raise}"/>
   </joint>
   <!-- ========== JOINT X : poutre Y qui glisse selon X (horizontale) ========== -->
@@ -84,5 +138,5 @@
     <parent link="base_link"/>
     <child link="gantry_y_beam"/>
-    <origin xyz="0 0 ${base_z + rail_x_h + beam_y_h/2}"/>
+    <origin xyz="0 0 ${base_z + rail_x_h + beam_y_h/2 + gantry_raise}"/>
     <axis xyz="1 0 0"/>
     <limit lower="${x_min}" upper="${x_max}" effort="80" velocity="0.4"/>
@@ -154,4 +208,7 @@
       <material name="black"/>
     </visual>
+    <collision>
+      <geometry><sphere radius="0.0015"/></geometry>
+    </collision>
   </link>
   <joint name="pen_tip_joint" type="fixed">
@@ -196,4 +253,11 @@
   </gazebo>
   <gazebo reference="base_link"><material>Gazebo/Grey</material></gazebo>
+  <gazebo reference="pcb_link">
+    <material>Gazebo/Green</material>
+    <mu1>0.4</mu1>
+    <mu2>0.4</mu2>
+    <kp>1000000.0</kp>
+    <kd>100.0</kd>
+  </gazebo>
   <gazebo reference="rail_x_pos"><material>Gazebo/Blue</material></gazebo>
   <gazebo reference="rail_x_neg"><material>Gazebo/Blue</material></gazebo>
@@ -208,3 +272,9 @@
     <kd>100.0</kd>
   </gazebo>
+  <gazebo reference="pen_tip">
+    <mu1>0.8</mu1>
+    <mu2>0.8</mu2>
+    <kp>1000000.0</kp>
+    <kd>100.0</kd>
+  </gazebo>
 </robot>

Commit message: fix(description): clean code src/drawbot_description/launch/display.launch.py src/drawbot_description/urdf/drawbot.urdf.xacro src/drawbot_description/CMakeLists.txt src/drawbot_description/package.xml

File: src/drawbot_description/urdf/drawbot.urdf.xacro (robot description, xacro)
@@ -253,6 +253,5 @@
   </gazebo>
   <gazebo reference="base_link"><material>Gazebo/Grey</material></gazebo>
-  <gazebo reference="pcb_link">
-    <material>Gazebo/Green</material>
+  <gazebo reference="pcb_link"><material>Gazebo/Green</material>
     <mu1>0.4</mu1>
     <mu2>0.4</mu2>

Commit message: refactor(geometry): centralize robot dimensions
Define shared mechanical dimensions and joint limits in a YAML configuration.

Load the same geometry from the Xacro model and Python control modules.

Document the shared configuration and declare its runtime dependencies.

File: src/drawbot_description/urdf/drawbot.urdf.xacro (robot description, xacro)
@@ -1,31 +1,32 @@
 <?xml version="1.0"?>
 <robot xmlns:xacro="http://www.ros.org/wiki/xacro" name="drawbot">
-  <!-- Géométrie (mètres) -->
-  <xacro:property name="base_x" value="0.36"/>
-  <xacro:property name="base_y" value="0.36"/>
-  <xacro:property name="base_z" value="0.020"/>
-  <xacro:property name="pcb_x" value="0.25"/>
-  <xacro:property name="pcb_y" value="0.25"/>
-  <xacro:property name="pcb_z" value="0.001"/>
+  <!-- Shared geometry (meters), also loaded by the Python control package. -->
+  <xacro:property name="geometry" value="${xacro.load_yaml('$(find drawbot_control)/config/drawbot_geometry.yaml')}"/>
+  <xacro:property name="base_x" value="${geometry['base']['x']}"/>
+  <xacro:property name="base_y" value="${geometry['base']['y']}"/>
+  <xacro:property name="base_z" value="${geometry['base']['thickness']}"/>
+  <xacro:property name="pcb_x" value="${geometry['pcb']['x']}"/>
+  <xacro:property name="pcb_y" value="${geometry['pcb']['y']}"/>
+  <xacro:property name="pcb_z" value="${geometry['pcb']['thickness']}"/>
   <!-- Raise the gantry so joint_pen=0 starts 7.5 mm above the PCB. -->
-  <xacro:property name="gantry_raise" value="0.0195"/>
-  <xacro:property name="support_size" value="0.020"/>
-  <xacro:property name="rail_x_len" value="0.32"/>
-  <xacro:property name="rail_x_w"   value="0.020"/>
-  <xacro:property name="rail_x_h"   value="0.020"/>
-  <xacro:property name="beam_y_len" value="0.32"/>
-  <xacro:property name="beam_y_w"   value="0.024"/>
-  <xacro:property name="beam_y_h"   value="0.024"/>
-  <xacro:property name="carriage_size" value="0.040"/>
-  <xacro:property name="pen_r" value="0.003"/>
-  <xacro:property name="pen_l" value="0.055"/>
+  <xacro:property name="gantry_raise" value="${geometry['gantry_raise']}"/>
+  <xacro:property name="support_size" value="${geometry['support']['size']}"/>
+  <xacro:property name="rail_x_len" value="${geometry['rail_x']['length']}"/>
+  <xacro:property name="rail_x_w"   value="${geometry['rail_x']['width']}"/>
+  <xacro:property name="rail_x_h"   value="${geometry['rail_x']['height']}"/>
+  <xacro:property name="beam_y_len" value="${geometry['beam_y']['length']}"/>
+  <xacro:property name="beam_y_w"   value="${geometry['beam_y']['width']}"/>
+  <xacro:property name="beam_y_h"   value="${geometry['beam_y']['height']}"/>
+  <xacro:property name="carriage_size" value="${geometry['carriage']['size']}"/>
+  <xacro:property name="pen_r" value="${geometry['pen']['radius']}"/>
+  <xacro:property name="pen_l" value="${geometry['pen']['length']}"/>
   <!-- Course -->
-  <xacro:property name="x_min" value="-0.10"/>
-  <xacro:property name="x_max" value="0.10"/>
-  <xacro:property name="y_min" value="-0.10"/>
-  <xacro:property name="y_max" value="0.10"/>
+  <xacro:property name="x_min" value="${geometry['limits']['x'][0]}"/>
+  <xacro:property name="x_max" value="${geometry['limits']['x'][1]}"/>
+  <xacro:property name="y_min" value="${geometry['limits']['y'][0]}"/>
+  <xacro:property name="y_max" value="${geometry['limits']['y'][1]}"/>
   <!-- Tip contact is near -6 mm; allow only 0.5 mm extra compression. -->
-  <xacro:property name="z_min" value="-0.0065"/>
-  <xacro:property name="z_max" value="0.020"/>
+  <xacro:property name="z_min" value="${geometry['limits']['z'][0]}"/>
+  <xacro:property name="z_max" value="${geometry['limits']['z'][1]}"/>
   <material name="grey"><color rgba="0.45 0.45 0.47 1"/></material>
   <material name="blue"><color rgba="0.12 0.35 0.85 1"/></material>
